File: pcb/hybridizer_manifold_interface/hybridizer_manifold_interface.sch (KiCad schematic (older format))
At the start: 17 parts, among them P1 HEADER_02X08_SMD

Commit message: Changes towards v1.1.
Parts:
- removed D1, D2, D3, D4, D5, D6, D7, D8: LED_24V_SMD, hybridizer_manifold_interface:LED_555-3XXX_SMD, symbol LED_24V_SMD
- removed P1: HEADER_02X08_SMD, hybridizer_manifold_interface:HEADER_02x08_SMD, symbol HEADER_02X08_SMD
- added C1, C11, C13, C15, C3, C5, C7, C9: 1uF, hybridizer_manifold_interface:SM0805_POL, symbol 1uF_0805_POL
- added C10, C12, C14, C16, C2, C4, C6, C8: 10nF, hybridizer_manifold_interface:SM0402, symbol 10nF_0402
- added D1, D2, D3, D4, D5, D6, D7, D8: diode_schottky_20V_1A, hybridizer_manifold_interface:SM0805_POL, symbol diode_schottky_20V_1A
- added P1: HEADER_02X07_SMD, hybridizer_manifold_interface:HEADER_02x07_SMD, symbol HEADER_02X07_SMD
- added R1, R11, R13, R15, R3, R5, R7, R9: 205k, hybridizer_manifold_interface:SM0402, symbol 205k_0402
- added R10, R12, R14, R16, R2, R4, R6, R8: 137k, hybridizer_manifold_interface:SM0402, symbol 137k_0402
- added U1, U2, U3, U4, U5, U6, U7, U8: DRV103, hybridizer_manifold_interface:SOIC_8, symbol DRV103
Connections:
- net OUT1 is gone; now on net GND: S2.2 (P2)
- net OUT2 is gone; now on net GND: S3.2 (P2)
- net OUT3 is gone; now on net GND: S4.2 (P2)
- net OUT4 is gone; now on net GND: S5.2 (P2)
- net OUT5 is gone; now on net GND: S6.2 (P2)
- net OUT6 is gone; now on net GND: S7.2 (P2)
- net OUT7 is gone; now on net GND: S8.2 (P2)
- net VAA: now also C1.1, C11.1, C13.1, C15.1, C3.1, C5.1, C7.1, C9.1, D1.1 (K), D2.1 (K), D3.1 (K), D4.1 (K), D5.1 (K), D6.1 (K), D7.1 (K), D8.1 (K), P1.1 (P1), P1.3 (P3), U1.6 (Vs), U2.6 (Vs), U3.6 (Vs), U4.6 (Vs), U5.6 (Vs), U6.6 (Vs), U7.6 (Vs), U8.6 (Vs); no longer S1.1 (P1), S2.1 (P1), S3.1 (P1), S4.1 (P1), S5.1 (P1), S6.1 (P1), S7.1 (P1), S8.1 (P1)
- net OUT0 renamed GND
- net GND: now also C1.2, C10.2, C11.2, C12.2, C13.2, C14.2, C15.2, C16.2, C2.2, C3.2, C4.2, C5.2, C6.2, C7.2, C8.2, C9.2, P1.2 (P2), P1.4 (P4), P1.6 (P6), R1.2, R10.2, R11.2, R12.2, R13.2, R14.2, R15.2, R16.2, R2.2, R3.2, R4.2, R5.2, R6.2, R7.2, R8.2, R9.2, U1.4 (GND), U2.4 (GND), U3.4 (GND), U4.4 (GND), U5.4 (GND), U6.4 (GND), U7.4 (GND), U8.4 (GND)
- new net: R2.1, U1.1 (DUTY)
- new net: C2.1, U1.2 (DELAY)
- new net: R1.1, U1.3 (FREQ)
- new net: R4.1, U2.1 (DUTY)
- new net: C4.1, U2.2 (DELAY)
- new net: R3.1, U2.3 (FREQ)
- new net: R6.1, U3.1 (DUTY)
- new net: C6.1, U3.2 (DELAY)
- new net: R5.1, U3.3 (FREQ)
- new net: R8.1, U4.1 (DUTY)
- new net: C8.1, U4.2 (DELAY)
- new net: R7.1, U4.3 (FREQ)
- new net: R10.1, U5.1 (DUTY)
- new net: C10.1, U5.2 (DELAY)
- new net: R9.1, U5.3 (FREQ)
- new net: R12.1, U6.1 (DUTY)
- new net: C12.1, U6.2 (DELAY)
- new net: R11.1, U6.3 (FREQ)
- new net: R14.1, U7.1 (DUTY)
- new net: C14.1, U7.2 (DELAY)
- new net: R13.1, U7.3 (FREQ)
- new net: R16.1, U8.1 (DUTY)
- new net: C16.1, U8.2 (DELAY)
- new net: R15.1, U8.3 (FREQ)
- new net IO0: P1.7 (P7), U1.8 (INPUT)
- new net IO1: P1.8 (P8), U2.8 (INPUT)
- new net IO2: P1.9 (P9), U3.8 (INPUT)
- new net IO3: P1.10 (P10), U4.8 (INPUT)
- new net IO4: P1.11 (P11), U5.8 (INPUT)
- new net IO5: P1.12 (P12), U6.8 (INPUT)
- new net IO6: P1.13 (P13), U7.8 (INPUT)
- new net IO7: P1.14 (P14), U8.8 (INPUT)
- new net SH0: D1.2 (A), S1.1 (P1), U1.5 (OUT)
- new net SH1: D2.2 (A), S2.1 (P1), U2.5 (OUT)
- new net SH2: D3.2 (A), S3.1 (P1), U3.5 (OUT)
- new net SH3: D4.2 (A), S4.1 (P1), U4.5 (OUT)
- new net SH4: D5.2 (A), S5.1 (P1), U5.5 (OUT)
- new net SH5: D6.2 (A), S6.1 (P1), U6.5 (OUT)
- new net SH6: D7.2 (A), S7.1 (P1), U7.5 (OUT)
- new net SH7: D8.2 (A), S8.1 (P1), U8.5 (OUT)
- no-connect marks 0 -> 9
