File: pcb/hybridizer_manifold_interface/hybridizer_manifold_interface.sch (KiCad schematic (older format))
At the start: 57 parts, among them P1 HEADER_02X07_SMD, U1 DRV103, U2 DRV103, U3 DRV103, U4 DRV103, U5 DRV103, U6 DRV103, U7 DRV103, U8 DRV103

Commit message: Finished hybridizer_manifold_interface_v1.1.
Parts:
- added D10, D11, D12, D13, D14, D15, D16, D9: LED_0805, hybridizer_manifold_interface:LED0805, symbol LED_0805
- added R17, R18, R19, R20, R21, R22, R23, R24: 300, hybridizer_manifold_interface:SM0402, symbol 300_0402
Connections:
- net GND: now also D10.2 (K), D11.2 (K), D12.2 (K), D13.2 (K), D14.2 (K), D15.2 (K), D16.2 (K), D9.2 (K)
- net IO0: now also R17.1
- net IO1: now also R18.1
- net IO2: now also R19.1
- net IO3: now also R20.1
- net IO4: now also R21.1
- net IO5: now also R22.1
- net IO6: now also R23.1
- net IO7: now also R24.1
- new net: D9.1 (A), R17.2
- new net: D10.1 (A), R18.2
- new net: D11.1 (A), R19.2
- new net: D12.1 (A), R20.2
- new net: D13.1 (A), R21.2
- new net: D14.1 (A), R22.2
- new net: D15.1 (A), R23.2
- new net: D16.1 (A), R24.2
Other:
- moved on the sheet: C1, C10, C11, C12, C13, C14, C15, C16, C2, C3, C4, C5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

Commit message: Initial changes to new version.
Connections:
- net GND: no longer S1.2 (P2), S2.2 (P2), S3.2 (P2), S4.2 (P2), S5.2 (P2), S6.2 (P2), S7.2 (P2), S8.2 (P2)
- net SH0: now also S1.2 (P2); no longer S1.1 (P1)
- net SH1: now also S2.2 (P2); no longer S2.1 (P1)
- net SH2: now also S3.2 (P2); no longer S3.1 (P1)
- net SH3: now also S4.2 (P2); no longer S4.1 (P1)
- net SH4: now also S5.2 (P2); no longer S5.1 (P1)
- net SH5: now also S6.2 (P2); no longer S6.1 (P1)
- net SH6: now also S7.2 (P2); no longer S7.1 (P1)
- net SH7: now also S8.2 (P2); no longer S8.1 (P1)
- net VAA: now also S1.1 (P1), S2.1 (P1), S3.1 (P1), S4.1 (P1), S5.1 (P1), S6.1 (P1), S7.1 (P1), S8.1 (P1)

Commit message: Made changes towards v1.2.
Parts:
- C1, C11, C13, C15, C3, C5, C7, C9: footprint hybridizer_manifold_interface:SM0805_POL -> hybridizer_manifold_interface:SM0805_POL_L
Connections:
- net at U1.1 (DUTY): now also R2.1; no longer C2.1
- net at U1.2 (DELAY): now also C2.1; no longer R1.1
- net at U1.3 (FREQ): now also R1.1; no longer R2.1
- net at U2.1 (DUTY): now also R4.1; no longer C4.1
- net at U2.2 (DELAY): now also C4.1; no longer R3.1
- net at U2.3 (FREQ): now also R3.1; no longer R4.1
- net at U3.1 (DUTY): now also R6.1; no longer C6.1
- net at U3.2 (DELAY): now also C6.1; no longer R5.1
- net at U3.3 (FREQ): now also R5.1; no longer R6.1
- net at U4.1 (DUTY): now also R8.1; no longer C8.1
- net at U4.2 (DELAY): now also C8.1; no longer R7.1
- net at U4.3 (FREQ): now also R7.1; no longer R8.1
- net at U5.1 (DUTY): now also R10.1; no longer C10.1
- net at U5.2 (DELAY): now also C10.1; no longer R9.1
- net at U5.3 (FREQ): now also R9.1; no longer R10.1
- net at U6.1 (DUTY): now also R12.1; no longer C12.1
- net at U6.2 (DELAY): now also C12.1; no longer R11.1
- net at U6.3 (FREQ): now also R11.1; no longer R12.1
- net at U7.1 (DUTY): now also R14.1; no longer C14.1
- net at U7.2 (DELAY): now also C14.1; no longer R13.1
- net at U7.3 (FREQ): now also R13.1; no longer R14.1
- net at U8.1 (DUTY): now also R16.1; no longer C16.1
- net at U8.2 (DELAY): now also C16.1; no longer R15.1
- net at U8.3 (FREQ): now also R15.1; no longer R16.1
Other:
- moved on the sheet: C10, C12, C14, C16, C2, C4, C6, C8, R1, R10, R11, R12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
