File: pcb/hybridizer_manifold_interface/hybridizer_manifold_interface.kicad_pcb (KiCad board)
At the start: 2 copper layers, 24 x 59.4 mm, 19 parts, among them P1 HEADER_02X08_SMD

Commit message: Changes towards v1.1.
Parts:
- removed MOUNTING_HOLE_0: mounting_hole, hybridizer_manifold_interface:mounting_hole
- added C1: 1uF, hybridizer_manifold_interface:SM0805_POL, B.Cu at (43.7, 29.7)
- added C10: 10nF, hybridizer_manifold_interface:SM0402, B.Cu at (36.7, 60.2)
- added C11: 1uF, hybridizer_manifold_interface:SM0805_POL, B.Cu at (43.7, 67.8)
- added C12: 10nF, hybridizer_manifold_interface:SM0402, B.Cu at (36.7, 67.8)
- added C13: 1uF, hybridizer_manifold_interface:SM0805_POL, B.Cu at (43.7, 75.4)
- added C14: 10nF, hybridizer_manifold_interface:SM0402, B.Cu at (36.7, 78.0)
- added C15: 1uF, hybridizer_manifold_interface:SM0805_POL, B.Cu at (43.7, 83.1)
- added C16: 10nF, hybridizer_manifold_interface:SM0402, B.Cu at (36.7, 83.1)
- added C2: 10nF, hybridizer_manifold_interface:SM0402, B.Cu at (36.7, 29.7)
- added C3: 1uF, hybridizer_manifold_interface:SM0805_POL, B.Cu at (43.7, 37.3)
- added C4: 10nF, hybridizer_manifold_interface:SM0402, B.Cu at (36.7, 39.9)
- added C5: 1uF, hybridizer_manifold_interface:SM0805_POL, B.Cu at (43.7, 45.0)
- added C6: 10nF, hybridizer_manifold_interface:SM0402, B.Cu at (36.7, 45.0)
- added C7: 1uF, hybridizer_manifold_interface:SM0805_POL, B.Cu at (43.7, 52.6)
- added C8: 10nF, hybridizer_manifold_interface:SM0402, B.Cu at (36.7, 52.6)
- added C9: 1uF, hybridizer_manifold_interface:SM0805_POL, B.Cu at (43.7, 60.2)
- added MOUNTING_HOLE_2: mounting_hole, hybridizer_manifold_interface:mounting_hole, F.Cu at (36.3, 74.2)
- added R1: 205k, hybridizer_manifold_interface:SM0402, B.Cu at (34.8, 29.7)
- added R10: 137k, hybridizer_manifold_interface:SM0402, B.Cu at (38.7, 60.2)
- added R11: 205k, hybridizer_manifold_interface:SM0402, B.Cu at (34.8, 67.8)
- added R12: 137k, hybridizer_manifold_interface:SM0402, B.Cu at (38.7, 67.8)
- added R13: 205k, hybridizer_manifold_interface:SM0402, B.Cu at (34.8, 78.0)
- added R14: 137k, hybridizer_manifold_interface:SM0402, B.Cu at (38.7, 78.0)
- added R15: 205k, hybridizer_manifold_interface:SM0402, B.Cu at (34.8, 83.1)
- added R16: 137k, hybridizer_manifold_interface:SM0402, B.Cu at (38.7, 83.1)
- added R2: 137k, hybridizer_manifold_interface:SM0402, B.Cu at (38.7, 29.7)
- added R3: 205k, hybridizer_manifold_interface:SM0402, B.Cu at (34.8, 39.9)
- added R4: 137k, hybridizer_manifold_interface:SM0402, B.Cu at (38.7, 39.9)
- added R5: 205k, hybridizer_manifold_interface:SM0402, B.Cu at (34.8, 45.0)
- added R6: 137k, hybridizer_manifold_interface:SM0402, B.Cu at (38.7, 45.0)
- added R7: 205k, hybridizer_manifold_interface:SM0402, B.Cu at (34.8, 52.6)
- added R8: 137k, hybridizer_manifold_interface:SM0402, B.Cu at (38.7, 52.6)
- added R9: 205k, hybridizer_manifold_interface:SM0402, B.Cu at (34.8, 60.2)
- added U1: DRV103, hybridizer_manifold_interface:SOIC_8, B.Cu at (29.8, 28.4)
- added U2: DRV103, hybridizer_manifold_interface:SOIC_8, B.Cu at (29.8, 36.1)
- added U3: DRV103, hybridizer_manifold_interface:SOIC_8, B.Cu at (29.8, 43.7)
- added U4: DRV103, hybridizer_manifold_interface:SOIC_8, B.Cu at (29.8, 51.3)
- added U5: DRV103, hybridizer_manifold_interface:SOIC_8, B.Cu at (29.8, 58.9)
- added U6: DRV103, hybridizer_manifold_interface:SOIC_8, B.Cu at (29.8, 66.5)
- added U7: DRV103, hybridizer_manifold_interface:SOIC_8, B.Cu at (29.8, 74.2)
- added U8: DRV103, hybridizer_manifold_interface:SOIC_8, B.Cu at (29.8, 81.8)
- D1, D2, D3, D4, D5, D6, D7, D8: value LED_24V_SMD -> diode_schottky_20V_1A; footprint hybridizer_manifold_interface:LED_555-3XXX_SMD -> hybridizer_manifold_interface:SM0805_POL; moved to B.Cu
- P1: value HEADER_02X08_SMD -> HEADER_02X07_SMD; footprint hybridizer_manifold_interface:HEADER_02x08_SMD -> hybridizer_manifold_interface:HEADER_02x07_SMD
- moved MOUNTING_HOLE_1 38.1 mm to (36.3, 36.1)
- moved D5 18.0 mm to (43.7, 57.7), turned to 0 degrees
- moved D6 18.0 mm to (43.7, 65.3), turned to 0 degrees
- moved D3 16.3 mm to (43.7, 42.4), turned to 0 degrees
- moved D4 16.3 mm to (43.7, 50.0), turned to 0 degrees
- moved D7 14.8 mm to (43.7, 72.9), turned to 0 degrees
- moved D2 13.7 mm to (43.7, 34.8), turned to 0 degrees
- moved D8 13.0 mm to (43.7, 80.5), turned to 0 degrees
- moved D1 12.7 mm to (43.7, 27.2), turned to 0 degrees
Connections:
- D1 pad 2: /OUT0 -> /SH0
- D2 pad 2: /OUT1 -> /SH1
- D3 pad 2: /OUT2 -> /SH2
- D4 pad 2: /OUT3 -> /SH3
- D5 pad 2: /OUT4 -> /SH4
- D6 pad 2: /OUT5 -> /SH5
- D7 pad 2: /OUT6 -> /SH6
- D8 pad 2: /OUT7 -> /SH7
- P1 pad 10: /OUT4 -> /IO3
- P1 pad 11: VAA -> /IO4
- P1 pad 12: /OUT5 -> /IO5
- P1 pad 13: VAA -> /IO6
- P1 pad 14: /OUT6 -> /IO7
- P1 pad 2: /OUT0 -> GND
- P1 pad 4: /OUT1 -> GND
- P1 pad 5: VAA -> Net-(P1-Pad5)
- P1 pad 6: /OUT2 -> GND
- P1 pad 7: VAA -> /IO0
- P1 pad 8: /OUT3 -> /IO1
- P1 pad 9: VAA -> /IO2
- S1 pad 1: VAA -> /SH0
- S1 pad 2: /OUT0 -> GND
- S2 pad 1: VAA -> /SH1
- S2 pad 2: /OUT1 -> GND
- S3 pad 1: VAA -> /SH2
- S3 pad 2: /OUT2 -> GND
- S4 pad 1: VAA -> /SH3
- S4 pad 2: /OUT3 -> GND
- S5 pad 1: VAA -> /SH4
- S5 pad 2: /OUT4 -> GND
- S6 pad 1: VAA -> /SH5
- S6 pad 2: /OUT5 -> GND
- S7 pad 1: VAA -> /SH6
- S7 pad 2: /OUT6 -> GND
- S8 pad 1: VAA -> /SH7
- S8 pad 2: /OUT7 -> GND
Routing:
- net VAA: track 137.8 -> 0.00 mm, vias 1 -> 0
- net /OUT1: track 44.4 -> 0.00 mm
- net /OUT6: track 39.8 -> 0.00 mm
- net /OUT4: track 38.8 -> 0.00 mm
- net /OUT0: track 38.5 -> 0.00 mm
- net /OUT7: track 37.1 -> 0.00 mm
- net /OUT2: track 33.2 -> 0.00 mm
- net /OUT5: track 32.7 -> 0.00 mm
- net /OUT3: track 31.5 -> 0.00 mm
- removed copper zone on B.Cu, net VAA
- removed copper zone on F.Cu, net VAA
Other:
- board text added: "hybridizer_manifold_interface Janelia Research Campus 05/2015 version 1.1 J005166"
- board text removed: "hybridizer_manifold_interface Janelia Research Campus 04/2015 version 1.0 J005166"

Commit message: Finished hybridizer_manifold_interface_v1.1.
Parts:
- added D10: LED_0805, hybridizer_manifold_interface:LED0805, F.Cu at (40.6, 36.1)
- added D11: LED_0805, hybridizer_manifold_interface:LED0805, F.Cu at (40.6, 43.7)
- added D12: LED_0805, hybridizer_manifold_interface:LED0805, F.Cu at (40.6, 51.3)
- added D13: LED_0805, hybridizer_manifold_interface:LED0805, F.Cu at (40.6, 58.9)
- added D14: LED_0805, hybridizer_manifold_interface:LED0805, F.Cu at (40.6, 66.5)
- added D15: LED_0805, hybridizer_manifold_interface:LED0805, F.Cu at (40.6, 74.2)
- added D16: LED_0805, hybridizer_manifold_interface:LED0805, F.Cu at (40.6, 81.8)
- added D9: LED_0805, hybridizer_manifold_interface:LED0805, F.Cu at (40.6, 28.4)
- added R17: 300, hybridizer_manifold_interface:SM0402, F.Cu at (40.6, 31.6)
- added R18: 300, hybridizer_manifold_interface:SM0402, F.Cu at (40.6, 39.2)
- added R19: 300, hybridizer_manifold_interface:SM0402, F.Cu at (40.6, 46.9)
- added R20: 300, hybridizer_manifold_interface:SM0402, F.Cu at (40.6, 54.5)
- added R21: 300, hybridizer_manifold_interface:SM0402, F.Cu at (40.6, 62.1)
- added R22: 300, hybridizer_manifold_interface:SM0402, F.Cu at (40.6, 69.7)
- added R23: 300, hybridizer_manifold_interface:SM0402, F.Cu at (40.6, 77.3)
- added R24: 300, hybridizer_manifold_interface:SM0402, F.Cu at (38.7, 81.8)
Routing:
- net GND: track 0.00 -> 241.6 mm, vias 0 -> 8
- net VAA: track 0.00 -> 182.1 mm, vias 0 -> 9
- net /IO0: track 0.00 -> 53.6 mm, vias 0 -> 1
- net /IO7: track 0.00 -> 40.7 mm, vias 0 -> 1
- net /IO1: track 0.00 -> 37.2 mm, vias 0 -> 1
- net /IO2: track 0.00 -> 34.3 mm, vias 0 -> 1
- net /SH4: track 0.00 -> 28.1 mm, vias 0 -> 2
- net /IO3: track 0.00 -> 28.1 mm, vias 0 -> 1
- net /SH3: track 0.00 -> 27.4 mm, vias 0 -> 1
- net /SH5: track 0.00 -> 27.3 mm, vias 0 -> 1
- net /SH2: track 0.00 -> 26.2 mm
- net /SH0: track 0.00 -> 25.5 mm, vias 0 -> 1
- net /IO6: track 0.00 -> 25.5 mm, vias 0 -> 1
- net /SH1: track 0.00 -> 25.3 mm
- net /SH6: track 0.00 -> 24.8 mm
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- added copper zone on F.Cu, net GND
- added copper zone on B.Cu, net VAA
Other:
- net class GND: trace_width 0.508 -> 0.8128
