File: pcb/hybridizer_manifold_interface/hybridizer_manifold_interface.kicad_pcb (KiCad board)
At the start: 2 copper layers, 24 x 59.4 mm, 75 parts, among them P1 HEADER_02X07_SMD, U1 DRV103, U2 DRV103, U3 DRV103, U4 DRV103, U5 DRV103, U6 DRV103, U7 DRV103, U8 DRV103

Commit message: Initial changes to new version.
Routing:
- net GND: track 241.6 -> 0.00 mm, vias 8 -> 0
- net VAA: track 182.1 -> 0.00 mm, vias 9 -> 0
- net /IO0: track 53.6 -> 0.00 mm, vias 1 -> 0
- net /IO7: track 40.7 -> 0.00 mm, vias 1 -> 0
- net /IO1: track 37.2 -> 0.00 mm, vias 1 -> 0
- net /IO2: track 34.3 -> 0.00 mm, vias 1 -> 0
- net /SH4: track 28.1 -> 0.00 mm, vias 2 -> 0
- net /IO3: track 28.1 -> 0.00 mm, vias 1 -> 0
- net /SH3: track 27.4 -> 0.00 mm, vias 1 -> 0
- net /SH5: track 27.3 -> 0.00 mm, vias 1 -> 0
- net /SH2: track 26.2 -> 0.00 mm
- net /SH0: track 25.5 -> 0.00 mm, vias 1 -> 0
- net /IO6: track 25.5 -> 0.00 mm, vias 1 -> 0
- net /SH1: track 25.3 -> 0.00 mm
- net /SH6: track 24.8 -> 0.00 mm
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- removed copper zone on F.Cu, net GND
- removed copper zone on B.Cu, net VAA

Commit message: Made changes towards v1.2.
Parts:
- C1, C11, C13, C15, C3, C5, C7, C9: footprint hybridizer_manifold_interface:SM0805_POL -> hybridizer_manifold_interface:SM0805_POL_L
- moved C15 1.98 mm to (42.2, 81.8), turned to 270 degrees
- moved C3 1.98 mm to (42.2, 36.1), turned to 270 degrees
- moved C7 1.98 mm to (42.2, 51.3), turned to 270 degrees
- moved C9 1.98 mm to (42.2, 58.9), turned to 270 degrees
- moved C1 1.98 mm to (42.2, 28.4), turned to 270 degrees
- moved C11 1.98 mm to (42.2, 66.5), turned to 270 degrees
- moved C13 1.98 mm to (42.2, 74.2), turned to 270 degrees
- moved C5 1.98 mm to (42.2, 43.7), turned to 270 degrees
- moved D7 1.80 mm to (45.0, 74.2), turned to 270 degrees
- moved D3 1.80 mm to (45.0, 43.7), turned to 270 degrees
- moved D4 1.80 mm to (45.0, 51.3), turned to 270 degrees
- moved D1 1.80 mm to (45.0, 28.4), turned to 270 degrees
- moved D2 1.80 mm to (45.0, 36.1), turned to 270 degrees
- moved D5 1.80 mm to (45.0, 58.9), turned to 270 degrees
- moved D6 1.80 mm to (45.0, 66.5), turned to 270 degrees
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Connections:
- S1 pad 1: /SH0 -> VAA
- S1 pad 2: GND -> /SH0
- S2 pad 1: /SH1 -> VAA
- S2 pad 2: GND -> /SH1
- S3 pad 1: /SH2 -> VAA
- S3 pad 2: GND -> /SH2
- S4 pad 1: /SH3 -> VAA
- S4 pad 2: GND -> /SH3
- S5 pad 1: /SH4 -> VAA
- S5 pad 2: GND -> /SH4
- S6 pad 1: /SH5 -> VAA
- S6 pad 2: GND -> /SH5
- S7 pad 1: /SH6 -> VAA
- S7 pad 2: GND -> /SH6
- S8 pad 1: /SH7 -> VAA
- S8 pad 2: GND -> /SH7
Routing:
- net GND: track 0.00 -> 5.08 mm
- net VAA: track 0.00 -> 2.54 mm
Other:
- net class GND: trace_width 0.8128 -> 0.6096
- net class POWER: trace_width 0.8128 -> 0.6096
- board text added: "hybridizer_manifold_interface Janelia Research Campus 06/2015 version 1.2 J005166"
- board text removed: "hybridizer_manifold_interface Janelia Research Campus 05/2015 version 1.1 J005166"

Commit message: Finished hybridizer_manifold_interface pcb v1.2.
Routing:
- net VAA: track 2.54 -> 299.4 mm
- net GND: track 5.08 -> 186.3 mm, vias 0 -> 7
- net /IO0: track 0.00 -> 42.7 mm, vias 0 -> 1
- net /IO6: track 0.00 -> 40.6 mm, vias 0 -> 1
- net /IO2: track 0.00 -> 40.0 mm, vias 0 -> 1
- net /IO1: track 0.00 -> 38.8 mm, vias 0 -> 1
- net /IO7: track 0.00 -> 31.3 mm, vias 0 -> 1
- net /IO3: track 0.00 -> 26.8 mm, vias 0 -> 1
- net /IO4: track 0.00 -> 25.7 mm, vias 0 -> 1
- net /IO5: track 0.00 -> 25.7 mm, vias 0 -> 1
- net /SH4: track 0.00 -> 25.4 mm
- net /SH6: track 0.00 -> 25.0 mm
- net /SH1: track 0.00 -> 24.9 mm
- net /SH7: track 0.00 -> 23.6 mm, vias 0 -> 1
- net /SH0: track 0.00 -> 22.6 mm
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- added copper zone on B.Cu, net GND
- added copper zone on F.Cu, net GND
- added copper zone on F.Cu, net VAA
Other:
- net class GND: trace_width 0.6096 -> 0.4064
- net class POWER: trace_width 0.6096 -> 0.4064
- net class SIGNAL: trace_width 0.4064 -> 0.254
