File: pcb/hybridizer_head_interface/hybridizer_head_interface.kicad_pcb (KiCad board)
At the start: 2 copper layers, 85.6 x 132.2 mm, 126 parts, among them P1 HEADER_02X07_SMD, P2 HEADER_02X05_SMD, P3 HEADER_02X05_SMD, U1 VA, U11 VA, U13 VA, U15 DRV103, U16 DRV103, U17 DRV103, U18 DRV103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

Commit message: Changes towards v1.3.
Parts:
- C22, C23, C24, C25, C30, C31, C32, C33: footprint hybridizer_head_interface:SM0805_POL -> hybridizer_head_interface:SM0805_POL_L
Routing:
- net GND: track 487.3 -> 401.4 mm, vias 7 -> 5
- net GNDA: track 390.6 -> 335.8 mm, vias 15 -> 12
- net /IO1: track 161.5 -> 114.7 mm, vias 0 -> 2
- net +5V: track 360.5 -> 396.9 mm, vias 16 -> 11
- net VAA: track 408.7 -> 430.6 mm, vias 0 -> 3
- net /A1: track 89.2 -> 74.6 mm
- net /IO5: track 76.5 -> 89.8 mm, vias 2 -> 0
- net /A0: track 73.8 -> 85.8 mm
- net /A2: track 45.4 -> 33.6 mm
- net /A12: track 65.8 -> 76.8 mm
- net /SH7: track 60.9 -> 49.9 mm, vias 1 -> 0
- net /A11: track 71.6 -> 81.3 mm
- net /IO7: track 63.2 -> 72.4 mm
- net /IO6: track 60.5 -> 55.0 mm
- net /A10: track 39.5 -> 34.9 mm
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- removed copper zone on F.Cu, net GND
- removed copper zone on B.Cu, net GNDA
Other:
- board text added: "A0-7"
- board text added: "A8-15"
- board text added: "IO0-7"
- board text added: "hybridizer_head_interface Janelia Research Campus 08/2015 version 1.3 J005165"
- board text removed: "hybridizer_head_interface Janelia Research Campus 06/2015 version 1.2 J005165"

Commit message: Updated hybridizer_head_interface to version 1.3.
Routing:
- net GNDA: track 335.8 -> 341.8 mm, vias 12 -> 13
- net GND: track 401.4 -> 407.0 mm, vias 5 -> 7
- added copper zone on F.Cu, net GND
- added copper zone on B.Cu, net GNDA
Changed lines of the file:
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@@
     (thickness 1.6)
     (drawings 31)
-    (tracks 1069)
+    (tracks 1078)
     (zones 0)
     (modules 126)
@@
   (segment (start 129.1776 88.434) (end 129.4508 88.1608) (width 0.4064) (layer F.Cu) (net 9))
   (segment (start 132.1562 88.0212) (end 129.4508 88.0212) (width 0.4064) (layer F.Cu) (net 9))
+  (segment (start 64.0258 41.66616) (end 63.119 41.66616) (width 0.508) (layer F.Cu) (net 10))
+  (via (at 66.294 41.03116) (size 0.889) (drill 0.635) (layers F.Cu B.Cu) (net 10))
+  (segment (start 62.484 41.03116) (end 66.294 41.03116) (width 0.508) (layer B.Cu) (net 10))
+  (via (at 62.484 41.03116) (size 0.889) (drill 0.635) (layers F.Cu B.Cu) (net 10))
+  (segment (start 63.119 41.66616) (end 62.484 41.03116) (width 0.508) (layer F.Cu) (net 10))
   (via (at 69.9843 88.0283) (size 0.889) (layers F.Cu B.Cu) (net 10))
   (via (at 91.2444 93.5955) (size 0.889) (layers F.Cu B.Cu) (net 10))
@@
   (segment (start 98.679 39.3116) (end 99.7658 39.3116) (width 0.508) (layer F.Cu) (net 10))
   (segment (start 88.519 50.3708) (end 86.614 50.3708) (width 0.508) (layer F.Cu) (net 10))
-  (segment (start 64.0258 43.7308) (end 64.0258 37.5437) (width 0.508) (layer F.Cu) (net 10))
+  (segment (start 64.0258 43.7308) (end 64.0258 41.66616) (width 0.508) (layer F.Cu) (net 10))
+  (segment (start 64.0258 41.66616) (end 64.0258 37.5437) (width 0.508) (layer F.Cu) (net 10))
   (segment (start 70.6658 50.3708) (end 64.0258 43.7308) (width 0.508) (layer F.Cu) (net 10))
   (segment (start 86.614 50.3708) (end 70.6658 50.3708) (width 0.508) (layer F.Cu) (net 10))
@@
   (segment (start 97.409 88.5038) (end 97.409 85.6072) (width 0.4064) (layer F.Cu) (net 60))
   (segment (start 94.6836 82.3062) (end 94.6836 83.0736) (width 0.4064) (layer F.Cu) (net 60))
+  (segment (start 76.2 34.6812) (end 76.2 31.88716) (width 0.508) (layer F.Cu) (net 69) (status 400000))
+  (via (at 73.914 29.60116) (size 0.889) (drill 0.635) (layers F.Cu B.Cu) (net 69))
+  (segment (start 76.2 31.88716) (end 73.914 29.60116) (width 0.508) (layer F.Cu) (net 69))
   (via (at 77.7572 71.3884) (size 0.889) (layers F.Cu B.Cu) (net 69))
   (via (at 109.2968 71.0743) (size 0.889) (layers F.Cu B.Cu) (net 69))
@@
   (segment (start 134.8616 74.8584) (end 123.7897 85.9303) (width 0.4064) (layer F.Cu) (net 78))
   (segment (start 134.8616 49.9212) (end 134.8616 74.8584) (width 0.4064) (layer F.Cu) (net 78))
+  (zone (net 10) (net_name GND) (layer F.Cu) (hatch edge 0.508)
+    (connect_pads (clearance 0.2032))
+    (min_thickness 0.2032)
+    (fill yes (arc_segments 16) (thermal_gap 0.508) (thermal_bridge_width 0.508))
+    (polygon
+      (pts
+        (xy 138.049 159.14116) (xy 49.784 159.14116) (xy 49.784 24.52116) (xy 138.049 24.52116) (xy 138.049 159.14116)
+      )
+    )
+  )
+  (zone (net 69) (net_name GNDA) (layer B.Cu) (hatch edge 0.508)
+    (connect_pads (clearance 0.2032))
+    (min_thickness 0.2032)
+    (fill yes (arc_segments 16) (thermal_gap 0.508) (thermal_bridge_width 0.508))
+    (polygon
+      (pts
+        (xy 138.684 159.77616) (xy 49.149 159.77616) (xy 49.149 23.88616) (xy 138.684 23.88616) (xy 138.684 159.77616)
+      )
+    )
+  )
 )
