File: pcb/hybridizer_head_interface/hybridizer_head_interface.sch (KiCad schematic (older format))
At the start: 60 parts, among them P1 HEADER_02X08_SMD, P2 HEADER_02X05_SMD, U1 HALL_DRV5053, U10 MAX4215, U11 HALL_DRV5053, U12 MAX4215, U13 HALL_DRV5053, U14 MAX4215, U2 MAX4215, U3 HALL_DRV5053, U4 MAX4215, U5 HALL_DRV5053, U6 MAX4215, U7 HALL_DRV5053, U8 MAX4215, U9 HALL_DRV5053

Commit message: Initial v1.1 changes.
Parts:
- added P10, P3, P4, P5, P6, P7, P8, P9: HEADER_01X03_SMD_F, hybridizer_head_interface:Header_3_Pin_SMD_F, symbol HEADER_01X03_SMD_F
- S1, S2, S3, S4, S5, S6, S7: Description CONN HEADER 2POS .100 VERT GOLD -> CONN BREAKAWAY SMD HDR 2POS; PartNumber 609-3500-ND -> WM9852-ND
Connections:
- net labels added: SH0, SH1, SH2, SH3, SH4, SH5, SH6, SH7
- wire segments 207 -> 232
Other:
- moved on the sheet: C1, C10, C11, C12, C13, C14, C15, C16, C17, C18, C19, C2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

Commit message: Made version 1.1 modifications.
Parts:
- removed P1: HEADER_02X08_SMD, hybridizer_head_interface:HEADER_02x08_SMD, symbol HEADER_02X08_SMD
- removed P10, P3, P4, P5, P6, P7, P8, P9: HEADER_01X03_SMD_F, hybridizer_head_interface:Header_3_Pin_SMD_F, symbol HEADER_01X03_SMD_F
- added P1: HEADER_02X07_SMD, hybridizer_head_interface:HEADER_02x07_SMD, symbol HEADER_02X07_SMD
Connections:
- net labels added: IO0, IO1, IO2, IO3, IO4, IO5, IO6, IO7
- net labels removed: OUT0, OUT1, OUT2, OUT3, OUT4, OUT5, OUT6, OUT7, SH0, SH1, SH2, SH3, SH4, SH5, SH6, SH7
- wire segments 232 -> 254
- no-connect marks 1 -> 3
Other:
- moved on the sheet: C10, C11, C12, C13, C14, C15, C16, C17, C18, C19, C20, C21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

Commit message: Changes towards v1.1.
Connections:
- net labels added: SH0, SH1, SH2, SH3, SH4, SH5, SH6, SH7
- wire segments 254 -> 209
Changed lines of the file:
@@
 	8950 4100 9150 4100
 Wire Wire Line
-	9150 3950 9150 4100
-Wire Wire Line
-	9150 4100 9150 4150
+	9150 3950 9150 4150
 Wire Wire Line
 	9150 3950 9250 3950
@@
 	8950 3600 9150 3600
 Wire Wire Line
-	9150 3550 9150 3600
-Wire Wire Line
-	9150 3600 9150 3750
+	9150 3550 9150 3750
 Wire Wire Line
 	9150 3750 9250 3750
@@
 	9650 3850 9800 3850
 Wire Wire Line
-	10300 3850 10500 3850
-Wire Wire Line
-	10500 3850 10950 3850
+	10300 3850 10950 3850
 Wire Wire Line
 	10500 3950 10500 3850
@@
 	10950 3950 10850 3950
 Wire Wire Line
-	10850 3950 10850 4050
-Wire Wire Line
-	10850 4050 10850 4150
+	10850 3950 10850 4150
 Wire Wire Line
 	10950 4050 10850 4050
@@
 	11850 4450 11850 4350
 Wire Wire Line
-	11850 3700 11850 3750
-Wire Wire Line
-	11850 3750 11850 3850
-Wire Wire Line
-	11850 3850 11850 3950
+	11850 3700 11850 3950
 Wire Wire Line
 	11550 3850 11850 3850
@@
 	8950 5400 9150 5400
 Wire Wire Line
-	9150 5250 9150 5400
-Wire Wire Line
-	9150 5400 9150 5450
+	9150 5250 9150 5450
 Wire Wire Line
 	9150 5250 9250 5250
@@
 	8950 4900 9150 4900
 Wire Wire Line
-	9150 4850 9150 4900
-Wire Wire Line
-	9150 4900 9150 5050
+	9150 4850 9150 5050
 Wire Wire Line
 	9150 5050 9250 5050
@@
 	9650 5150 9800 5150
 Wire Wire Line
-	10300 5150 10500 5150
-Wire Wire Line
-	10500 5150 10950 5150
+	10300 5150 10950 5150
 Wire Wire Line
 	10500 5250 10500 5150
@@
 	10950 5250 10850 5250
 Wire Wire Line
-	10850 5250 10850 5350
-Wire Wire Line
-	10850 5350 10850 5450
+	10850 5250 10850 5450
 Wire Wire Line
 	10950 5350 10850 5350
@@
 	11850 5750 11850 5650
 Wire Wire Line
-	11850 5000 11850 5050
-Wire Wire Line
-	11850 5050 11850 5150
-Wire Wire Line
-	11850 5150 11850 5250
+	11850 5000 11850 5250
 Wire Wire Line
 	11550 5150 11850 5150
@@
 	8950 6700 9150 6700
 Wire Wire Line
-	9150 6550 9150 6700
-Wire Wire Line
-	9150 6700 9150 6750
+	9150 6550 9150 6750
 Wire Wire Line
 	9150 6550 9250 6550
@@
 	8950 6200 9150 6200
 Wire Wire Line
-	9150 6150 9150 6200
-Wire Wire Line
-	9150 6200 9150 6350
+	9150 6150 9150 6350
 Wire Wire Line
 	9150 6350 9250 6350
@@
 	9650 6450 9800 6450
 Wire Wire Line
-	10300 6450 10500 6450
-Wire Wire Line
-	10500 6450 10950 6450
+	10300 6450 10950 6450
 Wire Wire Line
 	10500 6550 10500 6450
@@
 	10950 6550 10850 6550
 Wire Wire Line
-	10850 6550 10850 6650
-Wire Wire Line
-	10850 6650 10850 6750
+	10850 6550 10850 6750
 Wire Wire Line
 	10950 6650 10850 6650
@@
 	11850 7050 11850 6950
 Wire Wire Line
-	11850 6300 11850 6350
-Wire Wire Line
-	11850 6350 11850 6450
-Wire Wire Line
-	11850 6450 11850 6550
+	11850 6300 11850 6550
 Wire Wire Line
 	11550 6450 11850 6450
@@
 	8950 8000 9150 8000
 Wire Wire Line
-	9150 7850 9150 8000
-Wire Wire Line
-	9150 8000 9150 8050
+	9150 7850 9150 8050
 Wire Wire Line
 	9150 7850 9250 7850
@@
 	8950 7500 9150 7500
 Wire Wire Line
-	9150 7450 9150 7500
-Wire Wire Line
-	9150 7500 9150 7650
+	9150 7450 9150 7650
 Wire Wire Line
 	9150 7650 9250 7650
@@
 	9650 7750 9800 7750
 Wire Wire Line
-	10300 7750 10500 7750
-Wire Wire Line
-	10500 7750 10950 7750
+	10300 7750 10950 7750
 Wire Wire Line
 	10500 7850 10500 7750
@@
 	10950 7850 10850 7850
 Wire Wire Line
-	10850 7850 10850 7950
-Wire Wire Line
-	10850 7950 10850 8050
+	10850 7850 10850 8050
 Wire Wire Line
 	10950 7950 10850 7950
@@
 	11850 8350 11850 8250
 Wire Wire Line
-	11850 7600 11850 7650
-Wire Wire Line
-	11850 7650 11850 7750
-Wire Wire Line
-	11850 7750 11850 7850
+	11850 7600 11850 7850
 Wire Wire Line
 	11550 7750 11850 7750
@@
 	8950 9300 9150 9300
 Wire Wire Line
-	9150 9150 9150 9300
-Wire Wire Line
-	9150 9300 9150 9350
+	9150 9150 9150 9350
 Wire Wire Line
 	9150 9150 9250 9150
@@
 	8950 8800 9150 8800
 Wire Wire Line
-	9150 8750 9150 8800
-Wire Wire Line
-	9150 8800 9150 8950
+	9150 8750 9150 8950
 Wire Wire Line
 	9150 8950 9250 8950
@@
 	9650 9050 9800 9050
 Wire Wire Line
-	10300 9050 10500 9050
-Wire Wire Line
-	10500 9050 10950 9050
+	10300 9050 10950 9050
 Wire Wire Line
 	10500 9150 10500 9050
@@
 	10950 9150 10850 9150
 Wire Wire Line
-	10850 9150 10850 9250
-Wire Wire Line
-	10850 9250 10850 9350
+	10850 9150 10850 9350
 Wire Wire Line
 	10950 9250 10850 9250
@@
 	11850 9650 11850 9550
 Wire Wire Line
-	11850 8900 11850 8950
-Wire Wire Line
-	11850 8950 11850 9050
-Wire Wire Line
-	11850 9050 11850 9150
+	11850 8900 11850 9150
 Wire Wire Line
 	11550 9050 11850 9050
@@
 	12400 1250 12400 1350
 Wire Wire Line
-	12400 1350 12700 1350
-Wire Wire Line
-	12700 1350 12800 1350
+	12400 1350 12800 1350
 Wire Wire Line
 	12700 1250 12700 1350
@@
 	8950 2800 9150 2800
 Wire Wire Line
-	9150 2650 9150 2800
-Wire Wire Line
-	9150 2800 9150 2850
+	9150 2650 9150 2850
 Wire Wire Line
 	9150 2650 9250 2650
@@
 	8950 2300 9150 2300
 Wire Wire Line
-	9150 2250 9150 2300
-Wire Wire Line
-	9150 2300 9150 2450
+	9150 2250 9150 2450
 Wire Wire Line
 	9150 2450 9250 2450
@@
 	9650 2550 9800 2550
 Wire Wire Line
-	10300 2550 10500 2550
-Wire Wire Line
-	10500 2550 10950 2550
+	10300 2550 10950 2550
 Wire Wire Line
 	10500 2650 10500 2550
@@
 	10950 2650 10850 2650
 Wire Wire Line
-	10850 2650 10850 2750
-Wire Wire Line
-	10850 2750 10850 2850
+	10850 2650 10850 2850
 Wire Wire Line
 	10950 2750 10850 2750
@@
 	11850 3150 11850 3050
 Wire Wire Line
-	11850 2400 11850 2450
-Wire Wire Line
-	11850 2450 11850 2550
-Wire Wire Line
-	11850 2550 11850 2650
+	11850 2400 11850 2650
 Wire Wire Line
 	11550 2550 11850 2550
@@
 	8950 1500 9150 1500
 Wire Wire Line
-	9150 1350 9150 1500
-Wire Wire Line
-	9150 1500 9150 1550
+	9150 1350 9150 1550
 Wire Wire Line
 	9150 1350 9250 1350
@@
 	8950 1000 9150 1000
 Wire Wire Line
-	9150 950  9150 1000
-Wire Wire Line
-	9150 1000 9150 1150
+	9150 950  9150 1150
 Wire Wire Line
 	9150 1150 9250 1150
@@
 	9650 1250 9800 1250
 Wire Wire Line
-	10300 1250 10500 1250
-Wire Wire Line
-	10500 1250 10950 1250
+	10300 1250 10950 1250
 Wire Wire Line
 	10500 1350 10500 1250
@@
 	10950 1350 10850 1350
 Wire Wire Line
-	10850 1350 10850 1450
-Wire Wire Line
-	10850 1450 10850 1550
+	10850 1350 10850 1550
 Wire Wire Line
 	10950 1450 10850 1450
@@
 	11850 1850 11850 1750
 Wire Wire Line
-	11850 1100 11850 1150
-Wire Wire Line
-	11850 1150 11850 1250
-Wire Wire Line
-	11850 1250 11850 1350
+	11850 1100 11850 1350
 Wire Wire Line
 	11550 1250 11850 1250
@@
 $EndComp
 Wire Wire Line
-	5050 1350 5250 1350
-Wire Wire Line
-	5250 1350 5350 1350
-Wire Wire Line
-	5250 1350 5250 1250
-Wire Wire Line
-	5250 1250 5250 1150
+	5050 1350 5350 1350
+Wire Wire Line
+	5250 1150 5250 1350
 Wire Wire Line
 	5350 1250 5250 1250
@@
 IO7
 Wire Wire Line
-	5850 1250 6250 1250
-Wire Wire Line
-	6250 1250 6250 1350
-Wire Wire Line
-	6250 1350 6250 1450
-Wire Wire Line
-	6250 1450 6250 1500
+	5850 1250 6400 1250
+Wire Wire Line
+	6250 1250 6250 1500
 Wire Wire Line
 	5850 1450 6250 1450
@@
 Connection ~ 6250 1350
 Wire Wire Line
-	2150 1800 2500 1800
-Wire Wire Line
-	2500 1800 2850 1800
-Wire Wire Line
-	2850 1800 3200 1800
-Wire Wire Line
-	3200 1800 3350 1800
-Wire Wire Line
-	3350 1800 3550 1800
-Wire Wire Line
-	3550 1800 3900 1800
-Wire Wire Line
-	3900 1800 4250 1800
-Wire Wire Line
-	4250 1800 4600 1800
+	2150 1800 4600 1800
 Connection ~ 2500 1800
 Connection ~ 2850 1800
@@
 	1    0    0    -1
 $EndComp
+$Comp
+L PWR_FLAG #FLG?
+U 1 1 555370AA
+P 6400 1150
+F 0 "#FLG?" H 6400 1245 50  0001 C CNN
+F 1 "PWR_FLAG" H 6400 1330 50  0000 C CNN
+F 2 "" H 6400 1150 60  0000 C CNN
+F 3 "" H 6400 1150 60  0000 C CNN
+	1    6400 1150
+	1    0    0    -1
+$EndComp
+Wire Wire Line
+	6400 1250 6400 1150
+Connection ~ 6250 1250
+Wire Wire Line
+	1150 1000 950  1000
+Wire Wire Line
+	1150 1800 950  1800
+Wire Wire Line
+	1150 2600 950  2600
+Wire Wire Line
+	1150 3400 950  3400
+Wire Wire Line
+	1150 4200 950  4200
+Wire Wire Line
+	1150 5000 950  5000
+Wire Wire Line
+	1150 5800 950  5800
+Wire Wire Line
+	1150 6600 950  6600
+Text Label 950  1000 0    60   ~ 0
+SH0
+Text Label 950  1800 0    60   ~ 0
+SH1
+Text Label 950  2600 0    60   ~ 0
+SH2
+Text Label 950  3400 0    60   ~ 0
+SH3
+Text Label 950  4200 0    60   ~ 0
+SH4
+Text Label 950  5000 0    60   ~ 0
+SH5
+Text Label 950  5800 0    60   ~ 0
+SH6
+Text Label 950  6600 0    60   ~ 0
+SH7
 $EndSCHEMATC

Commit message: Progress towards hybridizer_head_interface_v1.1.
Parts:
- removed D1, D2, D3, D4, D5, D6, D7, D8: LED_24V_SMD, hybridizer_head_interface:LED_555-3XXX_SMD, symbol LED_24V_SMD
- added C22, C23, C24, C25, C30, C31, C32, C33: 1uF, hybridizer_head_interface:SM0805_POL, symbol 1uF_0805_POL
- added C26, C27, C28, C29, C34, C35, C36, C37: 10nF, hybridizer_head_interface:SM0402, symbol 10nF_0402
- added D1, D2, D3, D4, D5, D6, D7, D8: LED_0805, hybridizer_head_interface:LED0805, symbol LED_0805
- added D10, D11, D12, D13, D14, D15, D16, D9: diode_schottky_20V_1A, hybridizer_head_interface:SM0805_POL, symbol diode_schottky_20V_1A
- added R10, R11, R12, R13, R14, R15, R8, R9: 300, hybridizer_head_interface:SM0402, symbol 300_0402
- added R16, R18, R20, R22, R24, R26, R28, R30: 205k, hybridizer_head_interface:SM0402, symbol 205k_0402
- added R17, R19, R21, R23, R25, R27, R29: 110k, hybridizer_head_interface:SM0402, symbol 110k_0402
- added R31: 137k, hybridizer_head_interface:SM0402, symbol 137k_0402
- added U15, U16, U17, U18, U19, U20, U21, U22: DRV103, hybridizer_head_interface:SOIC_8, symbol DRV103
Connections:
- wire segments 209 -> 407
- no-connect marks 3 -> 11
Other:
- moved on the sheet: C1, C10, C11, C12, C13, C14, C15, C16, C17, C18, C19, C2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

Commit message: Finished hybridizer_head_interface pcb v1.1.
Parts:
- removed S1: HEADER_01X02_SMD, hybridizer_head_interface:Header_2_Pin_SMD, symbol HEADER_01X02_SMD
- removed U1, U11, U13, U3, U5, U7, U9: HALL_DRV5053, hybridizer_head_interface:SOT-23-3, symbol HALL_DRV5053
- added S1: HEADER_01X02_SMD_N, hybridizer_head_interface:Header_2_Pin_SMD_N, symbol HEADER_01X02_SMD_N
- added U1, U11, U13, U3, U5, U7, U9: HALL_DRV5053_OA_-73mT, hybridizer_head_interface:SOT-23-3, symbol HALL_DRV5053_OA_-73mT
Connections:
- net +5V: now also U1.1 (Vcc), U11.1 (Vcc), U13.1 (Vcc), U3.1 (Vcc), U5.1 (Vcc), U7.1 (Vcc), U9.1 (Vcc)
- net GND: now also S1.2 (P2), U1.3 (GND), U11.3 (GND), U13.3 (GND), U3.3 (GND), U5.3 (GND), U7.3 (GND), U9.3 (GND)
- net SH0: now also S1.1 (P1)
- net at R3.2: now also U5.2 (OUT)
- net at R4.2: now also U7.2 (OUT)
- net at R5.2: now also U9.2 (OUT)
- net at R6.2: now also U11.2 (OUT)
- net at R7.2: now also U13.2 (OUT)
- net at R2.2: now also U3.2 (OUT)
- net at R1.2: now also U1.2 (OUT)
Changed lines of the file:
@@
 NoConn ~ 14100 2150
-$Comp
-L HALL_DRV5053 U5
-U 1 1 5542A34F
-P 9450 3650
-F 0 "U5" H 9450 3450 40  0000 C CNN
-F 1 "HALL_DRV5053" H 9450 3850 40  0000 C CNN
-F 2 "hybridizer_head_interface:SOT-23-3" H 9350 3350 60  0001 C CNN
-F 3 "" H 9450 3650 60  0000 C CNN
-F 4 "digikey" H 9550 3550 60  0001 C CNN "Vendor"
-F 5 "296-38460-1-ND" H 9650 3650 60  0001 C CNN "PartNumber"
-F 6 "IC HALL SENSOR 9mT" H 9750 3750 60  0001 C CNN "Description"
-	1    9450 3650
-	1    0    0    -1
-$EndComp
-$Comp
-L HALL_DRV5053 U7
-U 1 1 5542A9A3
-P 9450 4950
-F 0 "U7" H 9450 4750 40  0000 C CNN
-F 1 "HALL_DRV5053" H 9450 5150 40  0000 C CNN
-F 2 "hybridizer_head_interface:SOT-23-3" H 9350 4650 60  0001 C CNN
-F 3 "" H 9450 4950 60  0000 C CNN
-F 4 "digikey" H 9550 4850 60  0001 C CNN "Vendor"
-F 5 "296-38460-1-ND" H 9650 4950 60  0001 C CNN "PartNumber"
-F 6 "IC HALL SENSOR 9mT" H 9750 5050 60  0001 C CNN "Description"
-	1    9450 4950
-	1    0    0    -1
-$EndComp
-$Comp
-L HALL_DRV5053 U9
-U 1 1 5542AA26
-P 9450 6250
-F 0 "U9" H 9450 6050 40  0000 C CNN
-F 1 "HALL_DRV5053" H 9450 6450 40  0000 C CNN
-F 2 "hybridizer_head_interface:SOT-23-3" H 9350 5950 60  0001 C CNN
-F 3 "" H 9450 6250 60  0000 C CNN
-F 4 "digikey" H 9550 6150 60  0001 C CNN "Vendor"
-F 5 "296-38460-1-ND" H 9650 6250 60  0001 C CNN "PartNumber"
-F 6 "IC HALL SENSOR 9mT" H 9750 6350 60  0001 C CNN "Description"
-	1    9450 6250
-	1    0    0    -1
-$EndComp
-$Comp
-L HALL_DRV5053 U11
-U 1 1 5542ABCE
-P 9450 7550
-F 0 "U11" H 9450 7350 40  0000 C CNN
-F 1 "HALL_DRV5053" H 9450 7750 40  0000 C CNN
-F 2 "hybridizer_head_interface:SOT-23-3" H 9350 7250 60  0001 C CNN
-F 3 "" H 9450 7550 60  0000 C CNN
-F 4 "digikey" H 9550 7450 60  0001 C CNN "Vendor"
-F 5 "296-38460-1-ND" H 9650 7550 60  0001 C CNN "PartNumber"
-F 6 "IC HALL SENSOR 9mT" H 9750 7650 60  0001 C CNN "Description"
-	1    9450 7550
-	1    0    0    -1
-$EndComp
-$Comp
-L HALL_DRV5053 U13
-U 1 1 5542AD5E
-P 9450 8850
-F 0 "U13" H 9450 8650 40  0000 C CNN
-F 1 "HALL_DRV5053" H 9450 9050 40  0000 C CNN
-F 2 "hybridizer_head_interface:SOT-23-3" H 9350 8550 60  0001 C CNN
-F 3 "" H 9450 8850 60  0000 C CNN
-F 4 "digikey" H 9550 8750 60  0001 C CNN "Vendor"
-F 5 "296-38460-1-ND" H 9650 8850 60  0001 C CNN "PartNumber"
-F 6 "IC HALL SENSOR 9mT" H 9750 8950 60  0001 C CNN "Description"
-	1    9450 8850
-	1    0    0    -1
-$EndComp
 $Comp
 L LEE_VALVE_PLUG_IN S8
@@
 F 6 "CONN RCPT PIN .025-.037in SOLDER" H 1650 7100 60  0001 C CNN "Description"
 	1    1350 6650
-	1    0    0    -1
-$EndComp
-$Comp
-L HEADER_01X02_SMD S1
-U 1 1 554B97B2
-P 1350 1050
-F 0 "S1" H 1350 1200 50  0000 C CNN
-F 1 "HEADER_01X02_SMD" V 1450 1050 50  0000 C CNN
-F 2 "hybridizer_head_interface:Header_2_Pin_SMD" H 1250 1100 60  0001 C CNN
-F 3 "" H 1350 1200 60  0000 C CNN
-F 4 "digikey" H 1450 1300 60  0001 C CNN "Vendor"
-F 5 "WM9852-ND" H 1550 1400 60  0001 C CNN "PartNumber"
-F 6 "CONN BREAKAWAY SMD HDR 2POS" H 1650 1500 60  0001 C CNN "Description"
-	1    1350 1050
 	1    0    0    -1
 $EndComp
@@
 $EndComp
 $Comp
-L HALL_DRV5053 U3
-U 1 1 554D7C92
-P 9450 2350
-F 0 "U3" H 9450 2150 40  0000 C CNN
-F 1 "HALL_DRV5053" H 9450 2550 40  0000 C CNN
-F 2 "hybridizer_head_interface:SOT-23-3" H 9350 2050 60  0001 C CNN
-F 3 "" H 9450 2350 60  0000 C CNN
-F 4 "digikey" H 9550 2250 60  0001 C CNN "Vendor"
-F 5 "296-38460-1-ND" H 9650 2350 60  0001 C CNN "PartNumber"
-F 6 "IC HALL SENSOR 9mT" H 9750 2450 60  0001 C CNN "Description"
-	1    9450 2350
-	1    0    0    -1
-$EndComp
-$Comp
 L 0.1uF C1
 U 1 1 554D7EE7
@@
 F 6 "IC OPAMP BUFFER 230MHZ RRO 8SOIC" H 11550 1150 60  0001 C CNN "Description"
 	1    11250 1100
-	1    0    0    -1
-$EndComp
-$Comp
-L HALL_DRV5053 U1
-U 1 1 554D7F53
-P 9450 1050
-F 0 "U1" H 9450 850 40  0000 C CNN
-F 1 "HALL_DRV5053" H 9450 1250 40  0000 C CNN
-F 2 "hybridizer_head_interface:SOT-23-3" H 9350 750 60  0001 C CNN
-F 3 "" H 9450 1050 60  0000 C CNN
-F 4 "digikey" H 9550 950 60  0001 C CNN "Vendor"
-F 5 "296-38460-1-ND" H 9650 1050 60  0001 C CNN "PartNumber"
-F 6 "IC HALL SENSOR 9mT" H 9750 1150 60  0001 C CNN "Description"
-	1    9450 1050
 	1    0    0    -1
 $EndComp
@@
 Connection ~ 6250 1400
 Wire Wire Line
-	1150 1100 1050 1100
-Wire Wire Line
-	1050 1100 1050 1200
+	1150 1050 1050 1050
+Wire Wire Line
+	1050 1050 1050 1150
 Wire Wire Line
 	1150 1900 1050 1900
@@
 L GND #PWR048
 U 1 1 554E77BF
-P 1050 1200
-F 0 "#PWR048" H 1050 950 50  0001 C CNN
-F 1 "GND" H 1050 1050 50  0000 C CNN
-F 2 "" H 1050 1200 60  0000 C CNN
-F 3 "" H 1050 1200 60  0000 C CNN
-	1    1050 1200
+P 1050 1150
+F 0 "#PWR048" H 1050 900 50  0001 C CNN
+F 1 "GND" H 1050 1000 50  0000 C CNN
+F 2 "" H 1050 1150 60  0000 C CNN
+F 3 "" H 1050 1150 60  0000 C CNN
+	1    1050 1150
 	1    0    0    -1
 $EndComp
@@
 Connection ~ 7250 1300
 Wire Wire Line
-	1150 1000 950  1000
+	1150 950  950  950
 Wire Wire Line
 	1150 1800 950  1800
@@
 Wire Wire Line
 	1150 6600 950  6600
-Text Label 950  1000 0    60   ~ 0
+Text Label 950  950  0    60   ~ 0
 SH0
 Text Label 950  1800 0    60   ~ 0
@@
 	1    0    0    -1
 $EndComp
+$Comp
+L HEADER_01X02_SMD_N S1
+U 1 1 555A0CF7
+P 1350 1000
+F 0 "S1" H 1350 1150 50  0000 C CNN
+F 1 "HEADER_01X02_SMD_N" V 1450 1000 50  0000 C CNN
+F 2 "hybridizer_head_interface:Header_2_Pin_SMD_N" H 1250 1050 60  0001 C CNN
+F 3 "" H 1350 1150 60  0000 C CNN
+F 4 "digikey" H 1450 1250 60  0001 C CNN "Vendor"
+F 5 "WM9852-ND" H 1550 1350 60  0001 C CNN "PartNumber"
+F 6 "CONN BREAKAWAY SMD HDR 2POS" H 1650 1450 60  0001 C CNN "Description"
+	1    1350 1000
+	1    0    0    -1
+$EndComp
+$Comp
+L HALL_DRV5053_OA_-73mT U1
+U 1 1 555A93A0
+P 9450 1050
+F 0 "U1" H 9450 850 40  0000 C CNN
+F 1 "HALL_DRV5053_OA_-73mT" H 9450 1250 40  0000 C CNN
+F 2 "hybridizer_head_interface:SOT-23-3" H 9350 750 60  0001 C CNN
+F 3 "" H 9450 850 60  0000 C CNN
+F 4 "digikey" H 9550 950 60  0001 C CNN "Vendor"
+F 5 "296-38457-1-ND" H 9650 1050 60  0001 C CNN "PartNumber"
+F 6 "IC HALL SENSOR OA -73mT" H 9750 1150 60  0001 C CNN "Description"
+	1    9450 1050
+	1    0    0    -1
+$EndComp
+$Comp
+L HALL_DRV5053_OA_-73mT U3
+U 1 1 555A9FB2
+P 9450 2350
+F 0 "U3" H 9450 2150 40  0000 C CNN
+F 1 "HALL_DRV5053_OA_-73mT" H 9450 2550 40  0000 C CNN
+F 2 "hybridizer_head_interface:SOT-23-3" H 9350 2050 60  0001 C CNN
+F 3 "" H 9450 2150 60  0000 C CNN
+F 4 "digikey" H 9550 2250 60  0001 C CNN "Vendor"
+F 5 "296-38457-1-ND" H 9650 2350 60  0001 C CNN "PartNumber"
+F 6 "IC HALL SENSOR OA -73mT" H 9750 2450 60  0001 C CNN "Description"
+	1    9450 2350
+	1    0    0    -1
+$EndComp
+$Comp
+L HALL_DRV5053_OA_-73mT U5
+U 1 1 555AA5D8
+P 9450 3650
+F 0 "U5" H 9450 3450 40  0000 C CNN
+F 1 "HALL_DRV5053_OA_-73mT" H 9450 3850 40  0000 C CNN
+F 2 "hybridizer_head_interface:SOT-23-3" H 9350 3350 60  0001 C CNN
+F 3 "" H 9450 3450 60  0000 C CNN
+F 4 "digikey" H 9550 3550 60  0001 C CNN "Vendor"
+F 5 "296-38457-1-ND" H 9650 3650 60  0001 C CNN "PartNumber"
+F 6 "IC HALL SENSOR OA -73mT" H 9750 3750 60  0001 C CNN "Description"
+	1    9450 3650
+	1    0    0    -1
+$EndComp
+$Comp
+L HALL_DRV5053_OA_-73mT U7
+U 1 1 555AAA96
+P 9450 4950
+F 0 "U7" H 9450 4750 40  0000 C CNN
+F 1 "HALL_DRV5053_OA_-73mT" H 9450 5150 40  0000 C CNN
+F 2 "hybridizer_head_interface:SOT-23-3" H 9350 4650 60  0001 C CNN
+F 3 "" H 9450 4750 60  0000 C CNN
+F 4 "digikey" H 9550 4850 60  0001 C CNN "Vendor"
+F 5 "296-38457-1-ND" H 9650 4950 60  0001 C CNN "PartNumber"
+F 6 "IC HALL SENSOR OA -73mT" H 9750 5050 60  0001 C CNN "Description"
+	1    9450 4950
+	1    0    0    -1
+$EndComp
+$Comp
+L HALL_DRV5053_OA_-73mT U9
+U 1 1 555AB208
+P 9450 6250
+F 0 "U9" H 9450 6050 40  0000 C CNN
+F 1 "HALL_DRV5053_OA_-73mT" H 9450 6450 40  0000 C CNN
+F 2 "hybridizer_head_interface:SOT-23-3" H 9350 5950 60  0001 C CNN
+F 3 "" H 9450 6050 60  0000 C CNN
+F 4 "digikey" H 9550 6150 60  0001 C CNN "Vendor"
+F 5 "296-38457-1-ND" H 9650 6250 60  0001 C CNN "PartNumber"
+F 6 "IC HALL SENSOR OA -73mT" H 9750 6350 60  0001 C CNN "Description"
+	1    9450 6250
+	1    0    0    -1
+$EndComp
+$Comp
+L HALL_DRV5053_OA_-73mT U11
+U 1 1 555AB6C2
+P 9450 7550
+F 0 "U11" H 9450 7350 40  0000 C CNN
+F 1 "HALL_DRV5053_OA_-73mT" H 9450 7750 40  0000 C CNN
+F 2 "hybridizer_head_interface:SOT-23-3" H 9350 7250 60  0001 C CNN
+F 3 "" H 9450 7350 60  0000 C CNN
+F 4 "digikey" H 9550 7450 60  0001 C CNN "Vendor"
+F 5 "296-38457-1-ND" H 9650 7550 60  0001 C CNN "PartNumber"
+F 6 "IC HALL SENSOR OA -73mT" H 9750 7650 60  0001 C CNN "Description"
+	1    9450 7550
+	1    0    0    -1
+$EndComp
+$Comp
+L HALL_DRV5053_OA_-73mT U13
+U 1 1 555ABB7E
+P 9450 8850
+F 0 "U13" H 9450 8650 40  0000 C CNN
+F 1 "HALL_DRV5053_OA_-73mT" H 9450 9050 40  0000 C CNN
+F 2 "hybridizer_head_interface:SOT-23-3" H 9350 8550 60  0001 C CNN
+F 3 "" H 9450 8650 60  0000 C CNN
+F 4 "digikey" H 9550 8750 60  0001 C CNN "Vendor"
+F 5 "296-38457-1-ND" H 9650 8850 60  0001 C CNN "PartNumber"
+F 6 "IC HALL SENSOR OA -73mT" H 9750 8950 60  0001 C CNN "Description"
+	1    9450 8850
+	1    0    0    -1
+$EndComp
